Commit message: added visual for chassis but still moves on its own

File: tfg_ws/src/track_model/models/xacro/deepracer/deepracer.urdf (robot description, URDF)
Before this commit: robot racecar, 12 links, 11 joints
Links:
- link chassis: geometry collision mesh filename=file://$(find track_model)/meshes/chassis.STL; visual mesh filename=file://$(find track_model)/meshes/chassis.STL

Commit message: fixed controller for deepracer, starting to tweak teleop

File: tfg_ws/src/track_model/models/xacro/deepracer/deepracer.urdf (robot description, URDF)
Before this commit: robot racecar, 12 links, 11 joints
Links:
- link shell: geometry collision mesh filename=file://$(find track_model)/meshes/deepracer_with_lidar.STL; visual mesh filename=file://$(find track_model)/meshes/deepracer_with_lidar.STL
